File: hardware/pcb/data_streamdeck.kicad_sch (KiCad schematic)
At the start: 19 parts, among them J1 KEY1 Top-Left, J2 KEY2 Top-Right, J3 KEY3 Mid-Left, J4 KEY4 Mid-Right, J5 KEY5 Bot-Left, J6 KEY6 Bot-Right, U1 ESP32-S3-DevKitC-1

Commit message: Rev E hardware, firmware 0.14.5, and docs for sensors and glow
Ship the dual-SPI carrier with IMU, ambient light, haptics, SK6812 edge
LEDs and Qwiic, plus companion flash overlay and GitHub Pages that match
the board.

Co-authored-by: Cursor <cursoragent@cursor.com>
Parts:
- removed U1: ESP32-S3-DevKitC-1, Module:ESP32-S3-DevKitC-1, symbol Connector_Generic:Conn_01x20
- added BZ1: CPT-9019S, Buzzer_Beeper:Buzzer_CUI_CPT-9019S-SMT, symbol Device:Buzzer
- added C10, C13, C14, C15, C16, C9: 100nF, Capacitor_SMD:C_0402_1005Metric, symbol Device:C
- added C11, C12: 1uF, Capacitor_SMD:C_0402_1005Metric, symbol Device:C
- added C17, C7, C8: 10uF, Capacitor_SMD:C_0805_2012Metric, symbol Device:C
- added D1: SK6812MINI-E (key J1), LED_SMD:LED_SK6812MINI_PLCC4_3.5x3.5mm_P1.75mm, symbol LED:SK6812
- added D2: SK6812MINI-E (key J2), LED_SMD:LED_SK6812MINI_PLCC4_3.5x3.5mm_P1.75mm, symbol LED:SK6812
- added D3: SK6812MINI-E (key J3), LED_SMD:LED_SK6812MINI_PLCC4_3.5x3.5mm_P1.75mm, symbol LED:SK6812
- added D4: SK6812MINI-E (key J4), LED_SMD:LED_SK6812MINI_PLCC4_3.5x3.5mm_P1.75mm, symbol LED:SK6812
- added D5: SK6812MINI-E (key J5), LED_SMD:LED_SK6812MINI_PLCC4_3.5x3.5mm_P1.75mm, symbol LED:SK6812
- added D6: SK6812MINI-E (key J6), LED_SMD:LED_SK6812MINI_PLCC4_3.5x3.5mm_P1.75mm, symbol LED:SK6812
- added D7: SK6812MINI-E (rear link), LED_SMD:LED_SK6812MINI_PLCC4_3.5x3.5mm_P1.75mm, symbol LED:SK6812
- added D8: SK6812MINI-E (rear SD), LED_SMD:LED_SK6812MINI_PLCC4_3.5x3.5mm_P1.75mm, symbol LED:SK6812
- added J10: LRA motor, Connector_JST:JST_SH_SM02B-SRSS-TB_1x02-1MP_P1.00mm_Horizontal, symbol Connector_Generic:Conn_01x02
- added J7: USB4105-GF-A, Connector_USB:USB_C_Receptacle_GCT_USB4105-xx-A_16P_TopMnt_Horizontal, symbol Connector:USB_C_Receptacle_USB2.0_16P
- added J8: microSD DM3D-SF, Connector_Card:microSD_HC_Hirose_DM3D-SF, symbol Connector:Micro_SD_Card
- added J9: Qwiic (JST-SH), Connector_JST:JST_SH_SM04B-SRSS-TB_1x04-1MP_P1.00mm_Horizontal, symbol Connector_Generic:Conn_01x04
- added R10: 100R, Resistor_SMD:R_0402_1005Metric, symbol Device:R
- added R7, R8: 5.1k, Resistor_SMD:R_0402_1005Metric, symbol Device:R
- added R9: 10k, Resistor_SMD:R_0402_1005Metric, symbol Device:R
- added SW1: BOOT, Button_Switch_SMD:SW_Push_1P1T_NO_CK_KMR2, symbol Switch:SW_Push
- added SW2: RESET, Button_Switch_SMD:SW_Push_1P1T_NO_CK_KMR2, symbol Switch:SW_Push
- added U1: ESP32-S3-WROOM-1-N16R8, RF_Module:ESP32-S3-WROOM-1, symbol RF_Module:ESP32-S3-WROOM-1
- added U2: AMS1117-3.3, Package_TO_SOT_SMD:SOT-223-3_TabPin2, symbol Regulator_Linear:AMS1117-3.3
- added U3: USBLC6-2SC6, Package_TO_SOT_SMD:SOT-23-6, symbol Power_Protection:USBLC6-2SC6
- added U4: LSM6DS3TR-C, Package_LGA:LGA-14_3x2.5mm_P0.5mm_LayoutBorder3x4y, symbol Sensor_Motion:LSM6DS3
- added U5: VEML7700, OpenScreenDeck:VEML7700-TT, symbol Connector_Generic:Conn_01x04
- added U6: DRV2605L, Package_SO:MSOP-10_3x3mm_P0.5mm, symbol Driver:DRV2605LDGS
- added U7: 74AHCT1G125, Package_TO_SOT_SMD:SOT-23-5, symbol 74xGxx:74AHCT1G125
- J1: value KEY1 Top-Left -> KEY1 Top-Left (bus A); footprint Connector_JST:JST_GH_SM09B-GHS-TB_1x09-1MP_P1.25mm_Horizontal -> Connector_Molex:Molex_PicoBlade_53261-0971_1x09-1MP_P1.25mm_Horizontal
- J2: value KEY2 Top-Right -> KEY2 Top-Right (bus A); footprint Connector_JST:JST_GH_SM09B-GHS-TB_1x09-1MP_P1.25mm_Horizontal -> Connector_Molex:Molex_PicoBlade_53261-0971_1x09-1MP_P1.25mm_Horizontal
- J3: value KEY3 Mid-Left -> KEY3 Mid-Left (bus A); footprint Connector_JST:JST_GH_SM09B-GHS-TB_1x09-1MP_P1.25mm_Horizontal -> Connector_Molex:Molex_PicoBlade_53261-0971_1x09-1MP_P1.25mm_Horizontal
- J4: value KEY4 Mid-Right -> KEY4 Mid-Right (bus B); footprint Connector_JST:JST_GH_SM09B-GHS-TB_1x09-1MP_P1.25mm_Horizontal -> Connector_Molex:Molex_PicoBlade_53261-0971_1x09-1MP_P1.25mm_Horizontal
- J5: value KEY5 Bot-Left -> KEY5 Bot-Left (bus B); footprint Connector_JST:JST_GH_SM09B-GHS-TB_1x09-1MP_P1.25mm_Horizontal -> Connector_Molex:Molex_PicoBlade_53261-0971_1x09-1MP_P1.25mm_Horizontal
- J6: value KEY6 Bot-Right -> KEY6 Bot-Right (bus B); footprint Connector_JST:JST_GH_SM09B-GHS-TB_1x09-1MP_P1.25mm_Horizontal -> Connector_Molex:Molex_PicoBlade_53261-0971_1x09-1MP_P1.25mm_Horizontal
Connections:
- net +3.3V: now also C1.1, C2.1, C3.1, C4.1, C5.1, C6.1, J1.7 (Pin_7), J2.7 (Pin_7), J3.7 (Pin_7), J4.7 (Pin_7), J5.7 (Pin_7), J6.7 (Pin_7), R1.1, R2.1, R3.1, R4.1, R5.1, R6.1, C10.1, C13.1, C14.1, C15.1, C7.1, C9.1, J8.4 (VDD), J9.2 (Pin_2), R9.1, U1.2 (3V3), U2.2 (VO), U4.12 (CS), U4.5 (VDDIO), U4.8 (VDD), U5.2 (Pin_2), U6.10 (VDD)
- net BL: now also J1.8 (Pin_8), J2.8 (Pin_8), J3.8 (Pin_8), J4.8 (Pin_8), J5.8 (Pin_8), J6.8 (Pin_8), U1.21 (IO13)
- net CS1: now also J1.3 (Pin_3), U1.18 (IO10)
- net CS2: now also J2.3 (Pin_3), U1.39 (IO1)
- net CS3: now also J3.3 (Pin_3), U1.38 (IO2)
- net CS4: now also J4.3 (Pin_3), U1.15 (IO3)
- net CS5: now also J5.3 (Pin_3), U1.4 (IO4)
- net CS6: now also J6.3 (Pin_3), U1.5 (IO5)
- net GND: now also C1.2, C2.2, C3.2, C4.2, C5.2, C6.2, J1.6 (Pin_6), J2.6 (Pin_6), J3.6 (Pin_6), J4.6 (Pin_6), J5.6 (Pin_6), J6.6 (Pin_6), BZ1.2 (-), C10.2, C11.2, C12.2, C13.2, C14.2, C15.2, C16.2, C17.2, C7.2, C8.2, C9.2, D1.1 (VSS), D2.1 (VSS), D3.1 (VSS), D4.1 (VSS), D5.1 (VSS), D6.1 (VSS), D7.1 (VSS), D8.1 (VSS), J7.A1 (GND), J7.A12 (GND), J7.B1 (GND), J7.B12 (GND), J7.SH (SHIELD), J8.6 (VSS), J8.SH (SHIELD), J9.1 (Pin_1), R7.2, R8.2, SW1.2, SW2.2, U1.1 (GND), U1.40 (GND), U1.41 (GND), U2.1 (GND), U3.2 (GND), U4.1 (SDO/SA0), U4.6 (GND), U4.7 (GND), U5.3 (Pin_3), U6.8 (GND), U7.1, U7.3 (GND)
- net KEY1: now also J1.1 (Pin_1), R1.2, U1.31 (IO38)
- net KEY2: now also J2.1 (Pin_1), R2.2, U1.32 (IO39)
- net KEY3: now also J3.1 (Pin_1), R3.2, U1.33 (IO40)
- net KEY4: now also J4.1 (Pin_1), R4.2, U1.34 (IO41)
- net KEY5: now also J5.1 (Pin_1), R5.2, U1.35 (IO42)
- net KEY6: now also J6.1 (Pin_1), R6.2, U1.24 (IO47)
- net RST: now also J1.9 (Pin_9), J2.9 (Pin_9), J3.9 (Pin_9), J4.9 (Pin_9), J5.9 (Pin_9), J6.9 (Pin_9), U1.23 (IO21)
- net DC_B: now reaches J6.2 (Pin_2)
- net DC_B: now also J4.2 (Pin_2), J5.2 (Pin_2), U1.12 (IO8)
- net SCK_B: now reaches J6.4 (Pin_4)
- net SCK_B: now also J4.4 (Pin_4), J5.4 (Pin_4), U1.11 (IO18)
- net MOSI_B: now reaches J6.5 (Pin_5)
- net MOSI_B: now also J4.5 (Pin_5), J5.5 (Pin_5), U1.10 (IO17)
- net DC_A: now reaches J3.2 (Pin_2)
- net DC_A: now also J1.2 (Pin_2), J2.2 (Pin_2), U1.22 (IO14)
- net SCK_A: now reaches J3.4 (Pin_4)
- net SCK_A: now also J1.4 (Pin_4), J2.4 (Pin_4), J8.5 (CLK), U1.20 (IO12)
- net MOSI_A: now reaches J3.5 (Pin_5)
- net MOSI_A: now also J1.5 (Pin_5), J2.5 (Pin_5), J8.3 (CMD), U1.19 (IO11)
- new net BOOT: SW1.1, U1.27 (IO0)
- new net CC1: J7.A5 (CC1), R7.1
- new net CC2: J7.B5 (CC2), R8.1
- new net DRV_REG: C12.1, U6.1 (REG)
- new net EN: C11.1, R9.2, SW2.1, U1.3 (EN)
- new net HAPTIC_EN: U1.36 (RXD0), U6.5 (EN)
- new net HAP_N: J10.2 (Pin_2), U6.9 (OUT-)
- new net HAP_P: J10.1 (Pin_1), U6.7 (OUT+)
- new net IMU_INT: U1.17 (IO9), U4.4 (INT1)
- new net LED_CH1: D7.2 (DIN), D8.4 (DOUT)
- new net LED_CH2: D2.4 (DOUT), D8.2 (DIN)
- new net LED_CH3: D2.2 (DIN), D4.4 (DOUT)
- new net LED_CH4: D4.2 (DIN), D6.4 (DOUT)
- new net LED_CH5: D5.4 (DOUT), D6.2 (DIN)
- new net LED_CH6: D3.4 (DOUT), D5.2 (DIN)
- new net LED_CH7: D1.4 (DOUT), D3.2 (DIN)
- new net LED_DATA_3V3: U1.25 (IO48), U7.2
- new net LED_DATA_5V: D7.4 (DOUT), U7.4
- new net MISO: J8.7 (DAT0), U1.8 (IO15)
- new net PIEZO: R10.1, U1.37 (TXD0)
- new net PIEZO_BZ: BZ1.1 (+), R10.2
- new net SCL: J9.4 (Pin_4), U1.7 (IO7), U4.13 (SCL), U5.1 (Pin_1), U6.2 (SCL)
- new net SDA: J9.3 (Pin_3), U1.6 (IO6), U4.14 (SDA), U5.4 (Pin_4), U6.3 (SDA)
- new net SD_CS: J8.2 (DAT3/CD), U1.9 (IO16)
- new net USB_D+: J7.A6 (D+), J7.B6 (D+), U1.14 (USB_D+), U3.1 (I/O1), U3.6 (I/O1)
- new net USB_D-: J7.A7 (D-), J7.B7 (D-), U1.13 (USB_D-), U3.3 (I/O2), U3.4 (I/O2)
- new net VBUS: C16.1, C17.1, C8.1, D1.3 (VDD), D2.3 (VDD), D3.3 (VDD), D4.3 (VDD), D5.3 (VDD), D6.3 (VDD), D7.3 (VDD), D8.3 (VDD), J7.A4 (VBUS), J7.A9 (VBUS), J7.B4 (VBUS), J7.B9 (VBUS), U2.3 (VI), U3.5 (VBUS), U7.5 (VCC)
- no-connect marks 0 -> 17
Other:
- note added: "Rev E — canonical pinout: hardware/pinout.py Regenerate: python3 scripts/generate_kicad_schematic.py"
- note removed: "Regenerate: python3 scripts/generate_kicad_schematic.py"
- company: Open Screen Deck -> LiteHawk Labs
- title: Open Screen Deck — 6-Key Carrier PCB -> Open Screen Deck — Rev E Carrier PCB
